File: pcb/ideal_diode.kicad_pcb (KiCad board)
At the start: 2 copper layers, 34 x 25 mm, 76 parts, among them P1 CONN_01X03, Q1 BSC028N06NS, Q2 BSC028N06NS, U1 LTC4359

Commit message: added title, date & version numbers to kicad schematic & pcb added *.kicad_pcb-bak *.bak *.net to git ignore
Parts:
- D1: value SMAT70A -> SMAJ60A
Changed lines of the file:
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@@
     (links 100)
     (no_connects 0)
-    (area 129.224999 88.724999 163.375001 113.875001)
+    (area 114.091667 85.472619 182.458334 122.775)
     (thickness 1.6)
     (drawings 9)
@@
   (page A4)
   (title_block
-    (title "20A Ideal Diode 4V-70V")
+    (title "20A Ideal Diode LTC4359 4V-70V")
+    (date 2016-01-22)
     (rev 1.0)
   )
   (layers
-    (0 F.Cu signal hide)
-    (31 B.Cu signal)
+    (0 F.Cu signal)
+    (31 B.Cu signal hide)
     (33 F.Adhes user)
     (35 F.Paste user)
@@
       (effects (font (size 1 1) (thickness 0.15)))
     )
-    (fp_text value SMAT70A (at 3.8 18.7 270) (layer F.Fab)
-      (effects (font (size 1 1) (thickness 0.15)))
-    )
+    (fp_text value SMAJ60A (at 3.8 18.7 270) (layer F.Fab)
+      (effects (font (size 1 1) (thickness 0.15)))
+    )
